Commit message: added main.py to simplify the code.

File: GEN3_URDF_V12_pybullet.urdf (robot description, URDF)
Before this commit: robot GEN3_URDF_V12, 9 links, 8 joints
Links:
- link Bracelet_Link: geometry collision mesh filename=C:/Users/udhay/Documents/Mtech(R)/Robot Manipulators/Assing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; visual mesh filename=C:/Users/udhay/Documents/Mtech(R)/Robot Manipulators/Assing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
- link ForeArm_Link: geometry collision mesh filename=C:/Users/udhay/Documents/Mtech(R)/Robot Manipulators/Assing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; visual mesh filename=C:/Users/udhay/Documents/Mtech(R)/Robot Manipulators/Assing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
- link HalfArm1_Link: geometry collision mesh filename=C:/Users/udhay/Documents/Mtech(R)/Robot Manipulators/Assing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; visual mesh filename=C:/Users/udhay/Documents/Mtech(R)/Robot Manipulators/Assing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
- link HalfArm2_Link: geometry collision mesh filename=C:/Users/udhay/Documents/Mtech(R)/Robot Manipulators/Assing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; visual mesh filename=C:/Users/udhay/Documents/Mtech(R)/Robot Manipulators/Assing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
- link Shoulder_Link: geometry collision mesh filename=C:/Users/udhay/Documents/Mtech(R)/Robot Manipulators/Assing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; visual mesh filename=C:/Users/udhay/Documents/Mtech(R)/Robot Manipulators/Assing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
- link SphericalWrist1_Link: geometry collision mesh filename=C:/Users/udhay/Documents/Mtech(R)/Robot Manipulators/Assing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; visual mesh filename=C:/Users/udhay/Documents/Mtech(R)/Robot Manipulators/Assing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
- link SphericalWrist2_Link: geometry collision mesh filename=C:/Users/udhay/Documents/Mtech(R)/Robot Manipulators/Assing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; visual mesh filename=C:/Users/udhay/Documents/Mtech(R)/Robot Manipulators/Assing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
- link base_link: geometry collision mesh filename=C:/Users/udhay/Documents/Mtech(R)/Robot Manipulators/Assing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; visual mesh filename=C:/Users/udhay/Documents/Mtech(R)/Robot Manipulators/Assing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

Commit message: added new main file.

File: GEN3_URDF_V12_pybullet.urdf (robot description, URDF)
Before this commit: robot GEN3_URDF_V12, 9 links, 8 joints
Links:
- link Bracelet_Link: geometry collision mesh filename=C:/Users/shash/OneDrive/Desktop/Subjects/RM_Assign/kinova_g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; visual mesh filename=C:/Users/shash/OneDrive/Desktop/Subjects/RM_Assign/kinova_g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
- link ForeArm_Link: geometry collision mesh filename=C:/Users/shash/OneDrive/Desktop/Subjects/RM_Assign/kinova_g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; visual mesh filename=C:/Users/shash/OneDrive/Desktop/Subjects/RM_Assign/kinova_g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
- link HalfArm1_Link: geometry collision mesh filename=C:/Users/shash/OneDrive/Desktop/Subjects/RM_Assign/kinova_g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; visual mesh filename=C:/Users/shash/OneDrive/Desktop/Subjects/RM_Assign/kinova_g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
- link HalfArm2_Link: geometry collision mesh filename=C:/Users/shash/OneDrive/Desktop/Subjects/RM_Assign/kinova_g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; visual mesh filename=C:/Users/shash/OneDrive/Desktop/Subjects/RM_Assign/kinova_g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
- link Shoulder_Link: geometry collision mesh filename=C:/Users/shash/OneDrive/Desktop/Subjects/RM_Assign/kinova_g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; visual mesh filename=C:/Users/shash/OneDrive/Desktop/Subjects/RM_Assign/kinova_g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
- link SphericalWrist1_Link: geometry collision mesh filename=C:/Users/shash/OneDrive/Desktop/Subjects/RM_Assign/kinova_g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; visual mesh filename=C:/Users/shash/OneDrive/Desktop/Subjects/RM_Assign/kinova_g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
- link SphericalWrist2_Link: geometry collision mesh filename=C:/Users/shash/OneDrive/Desktop/Subjects/RM_Assign/kinova_g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; visual mesh filename=C:/Users/shash/OneDrive/Desktop/Subjects/RM_Assign/kinova_g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
- link base_link: geometry collision mesh filename=C:/Users/shash/OneDrive/Desktop/Subjects/RM_Assign/kinova_g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; visual mesh filename=C:/Users/shash/OneDrive/Desktop/Subjects/RM_Assign/kinova_g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
